File: kicad/userport_expander.kicad_pcb (KiCad board)
At the start: 2 copper layers, 64.3 x 98 mm, 13 parts, among them J1 C64-UserPort, J2 Screw_Terminal_01x08, J3 Screw_Terminal_01x08, J4 Screw_Terminal_01x08, J5 Screw_Terminal_01x08, U1 4042, U2 8255

Commit message: added oshw logo
Parts:
- added REF***: OSHW-Logo_5.7x6mm_SilkScreen, Symbols:OSHW-Logo_5.7x6mm_SilkScreen, F.Cu at (128.2, 83.1)
Other:
- board text added: "©2019 Tulan"
